File: boards/pq-register/P1.kicad_sch (KiCad schematic)
At the start: 84 parts, among them Q1 T1-N652, Q10 T1-N652, Q102 T1-N652, Q103 T1-N652, Q11 T1-N652, Q2 T1-N652, Q3 T1-N652, Q4 T1-N652, Q5 T1-N652, Q6 T1-N652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

Commit message: Run ERC and clean up P & Q Register board.
Connections:
- net P1': now reaches Q4.3 (C), R65.1, R8.2
- net ~{P1'}: now reaches Q9.3 (C), R18.2, R84.2
- net P1a renamed P1b
- net Q renamed P1_{S}
- net ~{Q} renamed ~{P1_{S}}
Other:
- note added: "P1"
Changed lines of the file:
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@@
 		(title "LGP-21 P & Q Register Board")
 	)
+	(text "P1"
+		(exclude_from_sim no)
+		(at 166.37 40.64 0)
+		(effects
+			(font
+				(size 3.81 3.81)
+			)
+		)
+	)
 	(junction
 		(at 107.95 168.91)
@@
 			(width 0)
 			(type default)
+		)
+	)
+	(label "~{P1'}"
+		(at 196.85 67.31 0)
+		(effects
+			(font
+				(size 1.27 1.27)
+			)
+			(justify left bottom)
+		)
+	)
+	(label "P1'"
+		(at 133.35 67.31 0)
+		(effects
+			(font
+				(size 1.27 1.27)
+			)
+			(justify left bottom)
 		)
 	)
@@
 		)
 	)
-	(global_label "P1a"
+	(global_label "P1b"
 		(shape input)
 		(at 85.09 167.64 180)
@@
 		)
 	)
-	(hierarchical_label "~{Q}"
+	(hierarchical_label "~{P1_{S}}"
 		(shape output)
 		(at 214.63 30.48 0)
@@
 		)
 	)
-	(hierarchical_label "Q"
+	(hierarchical_label "P1_{S}"
 		(shape output)
 		(at 214.63 43.18 0)

Commit message: Add copyright information.
Other:
- company: (none) -> © 1962 General Precision; redrawn by Sam Hanes
Changed lines of the file:
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@@
 	(title_block
 		(title "LGP-21 P & Q Register Board")
+		(date "2026-06-15")
+		(rev "ESD 1060")
+		(company "© 1962 General Precision; redrawn by Sam Hanes")
+		(comment 1 "https://github.com/Elemecca/lgp21-docs")
 	)
 	(text "P1"
