File: boards/pq-register/P3.kicad_sch (KiCad schematic)
At the start: 36 parts, among them Q18 T1-N652, Q19 T1-N652, Q20 T1-N652, Q21 T1-N652, Q22 T1-N652, Q23 T1-N652

Commit message: Run ERC and clean up P & Q Register board.
Parts:
- renumbered C12 to C10, C16 to C12, C10 to C9
Connections:
- net ~{P3'}: now reaches Q21.3 (C), R108.2, R38.2
- net P3': now reaches Q19.3 (C), R103.1, R34.2
- net D renamed P2
- net P_{3} renamed P3
- net ~{D} renamed ~{P2}
- net ~{P_{3c}} renamed ~{P3c}
- net ~{P_{3d}} renamed ~{P3d}
- net ~{P_{3}} renamed ~{P3}
Other:
- note added: "P3"
Changed lines of the file:
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@@
 		(title "LGP-21 P & Q Register Board")
 	)
+	(text "P3"
+		(exclude_from_sim no)
+		(at 177.8 82.55 0)
+		(effects
+			(font
+				(size 3.81 3.81)
+			)
+		)
+	)
 	(junction
 		(at 152.4 85.09)
@@
 	)
 	(junction
+		(at 121.92 121.92)
+		(diameter 0)
+		(color 0 0 0 0)
+	)
+	(junction
 		(at 68.58 87.63)
 		(diameter 0)
@@
 	)
 	(junction
-		(at 214.63 85.09)
-		(diameter 0)
-		(color 0 0 0 0)
-	)
-	(junction
 		(at 187.96 92.71)
 		(diameter 0)
@@
 	)
 	(junction
-		(at 121.92 121.92)
-		(diameter 0)
-		(color 0 0 0 0)
-	)
-	(junction
 		(at 157.48 87.63)
 		(diameter 0)
@@
 	)
 	(junction
-		(at 214.63 63.5)
-		(diameter 0)
-		(color 0 0 0 0)
-	)
-	(junction
 		(at 121.92 74.93)
 		(diameter 0)
@@
 	(wire
 		(pts
-			(xy 214.63 90.17) (xy 214.63 85.09)
-		)
-		(stroke
-			(width 0)
-			(type default)
-		)
-	)
-	(wire
-		(pts
 			(xy 71.12 87.63) (xy 73.66 87.63)
 		)
@@
 	(wire
 		(pts
-			(xy 218.44 90.17) (xy 214.63 90.17)
-		)
-		(stroke
-			(width 0)
-			(type default)
-		)
-	)
-	(wire
-		(pts
 			(xy 71.12 132.08) (xy 71.12 129.54)
 		)
@@
 	(wire
 		(pts
-			(xy 208.28 109.22) (xy 208.28 121.92)
+			(xy 213.36 109.22) (xy 213.36 121.92)
 		)
 		(stroke
@@
 	(wire
 		(pts
-			(xy 214.63 68.58) (xy 214.63 63.5)
-		)
-		(stroke
-			(width 0)
-			(type default)
-		)
-	)
-	(wire
-		(pts
 			(xy 190.5 82.55) (xy 187.96 82.55)
 		)
@@
 	(wire
 		(pts
-			(xy 203.2 85.09) (xy 214.63 85.09)
+			(xy 203.2 85.09) (xy 218.44 85.09)
 		)
 		(stroke
@@
 	(wire
 		(pts
-			(xy 214.63 63.5) (xy 139.7 63.5)
+			(xy 139.7 63.5) (xy 218.44 63.5)
 		)
 		(stroke
@@
 	(wire
 		(pts
-			(xy 121.92 121.92) (xy 208.28 121.92)
+			(xy 121.92 121.92) (xy 213.36 121.92)
 		)
 		(stroke
@@
 	(wire
 		(pts
-			(xy 214.63 85.09) (xy 218.44 85.09)
-		)
-		(stroke
-			(width 0)
-			(type default)
-		)
-	)
-	(wire
-		(pts
-			(xy 218.44 68.58) (xy 214.63 68.58)
-		)
-		(stroke
-			(width 0)
-			(type default)
-		)
-	)
-	(wire
-		(pts
 			(xy 152.4 85.09) (xy 152.4 87.63)
 		)
@@
 	(wire
 		(pts
-			(xy 218.44 63.5) (xy 214.63 63.5)
-		)
-		(stroke
-			(width 0)
-			(type default)
-		)
-	)
-	(wire
-		(pts
 			(xy 203.2 83.82) (xy 203.2 85.09)
 		)
@@
 	(wire
 		(pts
-			(xy 205.74 109.22) (xy 208.28 109.22)
+			(xy 205.74 109.22) (xy 213.36 109.22)
 		)
 		(stroke
@@
 		)
 	)
+	(label "~{P3'}"
+		(at 208.28 109.22 0)
+		(effects
+			(font
+				(size 1.27 1.27)
+			)
+			(justify left bottom)
+		)
+	)
+	(label "P3'"
+		(at 144.78 109.22 0)
+		(effects
+			(font
+				(size 1.27 1.27)
+			)
+			(justify left bottom)
+		)
+	)
 	(global_label "i"
 		(shape input)
@@
 		)
 	)
-	(global_label "~{P_{3c}}"
+	(global_label "~{P3c}"
 		(shape input)
 		(at 100.33 76.2 180)
@@
 		)
 		(property "Intersheetrefs" "${INTERSHEET_REFS}"
-			(at 94.1855 76.2 0)
+			(at 93.7767 76.2 0)
 			(hide yes)
 			(show_name no)
@@
 		)
 	)
-	(global_label "~{P_{3}}"
+	(global_label "~{P3}"
 		(shape output)
 		(at 218.44 63.5 0)
@@
 		)
 		(property "Intersheetrefs" "${INTERSHEET_REFS}"
-			(at 223.7136 63.5 0)
+			(at 223.9047 63.5 0)
 			(hide yes)
 			(show_name no)
@@
 		)
 	)
-	(global_label "P_{3}"
-		(shape output)
-		(at 218.44 85.09 0)
+	(global_label "~{P2}"
+		(shape input)
+		(at 59.69 129.54 180)
 		(fields_autoplaced yes)
 		(effects
@@
 				(size 1.27 1.27)
 			)
-			(justify left)
+			(justify right)
 		)
 		(property "Intersheetrefs" "${INTERSHEET_REFS}"
-			(at 223.7136 85.09 0)
+			(at 54.2253 129.54 0)
 			(hide yes)
 			(show_name no)
@@
 					(size 1.27 1.27)
 				)
-				(justify left)
+				(justify right)
 			)
 		)
 	)
-	(global_label "~{P_{3d}}"
+	(global_label "P2"
 		(shape input)
-		(at 100.33 128.27 180)
+		(at 59.69 87.63 180)
 		(fields_autoplaced yes)
 		(effects
@@
 		)
 		(property "Intersheetrefs" "${INTERSHEET_REFS}"
-			(at 94.1372 128.27 0)
+			(at 54.2253 87.63 0)
 			(hide yes)
 			(show_name no)
@@
 		)
 	)
-	(hierarchical_label "Q"
+	(global_label "P3"
 		(shape output)
-		(at 218.44 90.17 0)
+		(at 218.44 85.09 0)
+		(fields_autoplaced yes)
 		(effects
 			(font
@@
 			(justify left)
 		)
-	)
-	(hierarchical_label "~{Q}"
-		(shape output)
-		(at 218.44 68.58 0)
-		(effects
-			(font
-				(size 1.27 1.27)
+		(property "Intersheetrefs" "${INTERSHEET_REFS}"
+			(at 223.9047 85.09 0)
+			(hide yes)
+			(show_name no)
+			(do_not_autoplace no)
+			(effects
+				(font
+					(size 1.27 1.27)
+				)
+				(justify left)
 			)
-			(justify left)
 		)
 	)
-	(hierarchical_label "D"
+	(global_label "~{P3d}"
 		(shape input)
-		(at 59.69 87.63 180)
+		(at 100.33 128.27 180)
+		(fields_autoplaced yes)
 		(effects
 			(font
@@
 			(justify right)
 		)
-	)
-	(hierarchical_label "~{D}"
-		(shape input)
-		(at 59.69 129.54 180)
-		(effects
-			(font
-				(size 1.27 1.27)
+		(property "Intersheetrefs" "${INTERSHEET_REFS}"
+			(at 93.7163 128.27 0)
+			(hide yes)
+			(show_name no)
+			(do_not_autoplace no)
+			(effects
+				(font
+					(size 1.27 1.27)
+				)
+				(justify right)
 			)
-			(justify right)
 		)
 	)
@@
 		(in_pos_files yes)
 		(dnp no)
-		(property "Reference" "C10"
+		(property "Reference" "C9"
 			(at 167.894 81.534 90)
 			(show_name no)
@@
 			(project "pq-register"
 				(path "/d5da316c-1ec9-4d99-8330-1c4a3f6c3ba4/d17b2d0e-6ffc-4e5b-aa1e-f1f6863801f5"
-					(reference "C10")
+					(reference "C9")
 					(unit 1)
 				)
@@
 		(in_pos_files yes)
 		(dnp no)
-		(property "Reference" "C16"
+		(property "Reference" "C12"
 			(at 198.374 81.534 90)
 			(show_name no)
@@
 			(project "pq-register"
 				(path "/d5da316c-1ec9-4d99-8330-1c4a3f6c3ba4/d17b2d0e-6ffc-4e5b-aa1e-f1f6863801f5"
-					(reference "C16")
+					(reference "C12")
 					(unit 1)
 				)
@@
 		(in_pos_files yes)
 		(dnp no)
-		(property "Reference" "C12"
+		(property "Reference" "C10"
 			(at 182.88 112.268 90)
 			(show_name no)
@@
 			(project "pq-register"
 				(path "/d5da316c-1ec9-4d99-8330-1c4a3f6c3ba4/d17b2d0e-6ffc-4e5b-aa1e-f1f6863801f5"
-					(reference "C12")
+					(reference "C10")
 					(unit 1)
 				)

Commit message: Add copyright information.
Other:
- company: (none) -> © 1962 General Precision; redrawn by Sam Hanes
Changed lines of the file:
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@@
 	(title_block
 		(title "LGP-21 P & Q Register Board")
+		(date "2026-06-15")
+		(rev "ESD 1060")
+		(company "© 1962 General Precision; redrawn by Sam Hanes")
+		(comment 1 "https://github.com/Elemecca/lgp21-docs")
 	)
 	(text "P3"
