File: boards/pq-register/P4.kicad_sch (KiCad schematic)
At the start: 36 parts, among them Q24 T1-N652, Q25 T1-N652, Q26 T1-N652, Q27 T1-N652, Q28 T1-N652, Q29 T1-N652

Commit message: Run ERC and clean up P & Q Register board.
Parts:
- renumbered C17 to C16
Connections:
- net P4': now reaches Q25.3 (C), R115.1, R44.2
- net ~{P4'}: now reaches Q27.3 (C), R120.2, R48.2
- net D renamed P3
- net P_{4} renamed P4
- net ~{D} renamed ~{P3}
- net ~{P_{4c}} renamed ~{P4c}
- net ~{P_{4d}} renamed ~{P4d}
- net ~{P_{4}} renamed ~{P4}
Other:
- note added: "P4"
Changed lines of the file:
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@@
 		(title "LGP-21 P & Q Register Board")
 	)
+	(text "P4"
+		(exclude_from_sim no)
+		(at 177.8 82.55 0)
+		(effects
+			(font
+				(size 3.81 3.81)
+			)
+		)
+	)
 	(junction
 		(at 167.64 92.71)
@@
 	)
 	(junction
-		(at 121.92 121.92)
-		(diameter 0)
-		(color 0 0 0 0)
-	)
-	(junction
-		(at 214.63 85.09)
-		(diameter 0)
-		(color 0 0 0 0)
-	)
-	(junction
 		(at 187.96 87.63)
 		(diameter 0)
@@
 	)
 	(junction
-		(at 214.63 63.5)
-		(diameter 0)
-		(color 0 0 0 0)
-	)
-	(junction
 		(at 177.8 109.22)
 		(diameter 0)
@@
 	)
 	(junction
+		(at 121.92 121.92)
+		(diameter 0)
+		(color 0 0 0 0)
+	)
+	(junction
 		(at 167.64 109.22)
 		(diameter 0)
@@
 	(wire
 		(pts
-			(xy 214.63 90.17) (xy 214.63 85.09)
-		)
-		(stroke
-			(width 0)
-			(type default)
-		)
-	)
-	(wire
-		(pts
 			(xy 121.92 120.65) (xy 121.92 121.92)
 		)
@@
 	(wire
 		(pts
-			(xy 218.44 90.17) (xy 214.63 90.17)
-		)
-		(stroke
-			(width 0)
-			(type default)
-		)
-	)
-	(wire
-		(pts
 			(xy 166.37 87.63) (xy 167.64 87.63)
 		)
@@
 	(wire
 		(pts
-			(xy 203.2 85.09) (xy 214.63 85.09)
-		)
-		(stroke
-			(width 0)
-			(type default)
-		)
-	)
-	(wire
-		(pts
 			(xy 121.92 121.92) (xy 121.92 123.19)
 		)
@@
 	(wire
 		(pts
-			(xy 121.92 121.92) (xy 208.28 121.92)
+			(xy 121.92 121.92) (xy 213.36 121.92)
 		)
 		(stroke
@@
 	(wire
 		(pts
-			(xy 205.74 109.22) (xy 208.28 109.22)
+			(xy 205.74 109.22) (xy 213.36 109.22)
 		)
 		(stroke
@@
 	(wire
 		(pts
-			(xy 214.63 68.58) (xy 214.63 63.5)
-		)
-		(stroke
-			(width 0)
-			(type default)
-		)
-	)
-	(wire
-		(pts
 			(xy 203.2 85.09) (xy 203.2 87.63)
 		)
@@
 	(wire
 		(pts
-			(xy 208.28 109.22) (xy 208.28 121.92)
+			(xy 213.36 109.22) (xy 213.36 121.92)
 		)
 		(stroke
@@
 	(wire
 		(pts
-			(xy 218.44 68.58) (xy 214.63 68.58)
-		)
-		(stroke
-			(width 0)
-			(type default)
-		)
-	)
-	(wire
-		(pts
-			(xy 214.63 85.09) (xy 218.44 85.09)
+			(xy 203.2 85.09) (xy 218.44 85.09)
 		)
 		(stroke
@@
 	(wire
 		(pts
-			(xy 218.44 63.5) (xy 214.63 63.5)
-		)
-		(stroke
-			(width 0)
-			(type default)
-		)
-	)
-	(wire
-		(pts
 			(xy 198.12 87.63) (xy 203.2 87.63)
 		)
@@
 	(wire
 		(pts
-			(xy 214.63 63.5) (xy 139.7 63.5)
+			(xy 139.7 63.5) (xy 218.44 63.5)
 		)
 		(stroke
@@
 		)
 	)
-	(global_label "P_{4}"
+	(label "~{P4'}"
+		(at 208.28 109.22 0)
+		(effects
+			(font
+				(size 1.27 1.27)
+			)
+			(justify left bottom)
+		)
+	)
+	(label "P4'"
+		(at 144.78 109.22 0)
+		(effects
+			(font
+				(size 1.27 1.27)
+			)
+			(justify left bottom)
+		)
+	)
+	(global_label "P4"
 		(shape output)
 		(at 218.44 85.09 0)
@@
 		)
 		(property "Intersheetrefs" "${INTERSHEET_REFS}"
-			(at 223.7136 85.09 0)
+			(at 223.9047 85.09 0)
 			(hide yes)
 			(show_name no)
@@
 		)
 	)
-	(global_label "~{P_{4c}}"
+	(global_label "~{P4c}"
 		(shape input)
 		(at 100.33 76.2 180)
@@
 		)
 		(property "Intersheetrefs" "${INTERSHEET_REFS}"
-			(at 94.1855 76.2 0)
+			(at 93.7767 76.2 0)
 			(hide yes)
 			(show_name no)
@@
 		)
 	)
-	(global_label "~{P_{4}}"
+	(global_label "~{P4}"
 		(shape output)
 		(at 218.44 63.5 0)
@@
 		)
 		(property "Intersheetrefs" "${INTERSHEET_REFS}"
-			(at 223.7136 63.5 0)
+			(at 223.9047 63.5 0)
 			(hide yes)
 			(show_name no)
@@
 		)
 	)
-	(global_label "~{P_{4d}}"
+	(global_label "~{P3}"
 		(shape input)
-		(at 100.33 128.27 180)
+		(at 59.69 129.54 180)
 		(fields_autoplaced yes)
 		(effects
@@
 		)
 		(property "Intersheetrefs" "${INTERSHEET_REFS}"
-			(at 94.1372 128.27 0)
+			(at 54.2253 129.54 0)
 			(hide yes)
 			(show_name no)
@@
 		)
 	)
-	(hierarchical_label "D"
+	(global_label "P3"
 		(shape input)
 		(at 59.69 87.63 180)
+		(fields_autoplaced yes)
 		(effects
 			(font
@@
 			(justify right)
 		)
-	)
-	(hierarchical_label "~{D}"
-		(shape input)
-		(at 59.69 129.54 180)
-		(effects
-			(font
-				(size 1.27 1.27)
+		(property "Intersheetrefs" "${INTERSHEET_REFS}"
+			(at 54.2253 87.63 0)
+			(hide yes)
+			(show_name no)
+			(do_not_autoplace no)
+			(effects
+				(font
+					(size 1.27 1.27)
+				)
+				(justify right)
 			)
-			(justify right)
 		)
 	)
-	(hierarchical_label "~{Q}"
-		(shape output)
-		(at 218.44 68.58 0)
+	(global_label "~{P4d}"
+		(shape input)
+		(at 100.33 128.27 180)
+		(fields_autoplaced yes)
 		(effects
 			(font
 				(size 1.27 1.27)
 			)
-			(justify left)
+			(justify right)
 		)
-	)
-	(hierarchical_label "Q"
-		(shape output)
-		(at 218.44 90.17 0)
-		(effects
-			(font
-				(size 1.27 1.27)
+		(property "Intersheetrefs" "${INTERSHEET_REFS}"
+			(at 93.7163 128.27 0)
+			(hide yes)
+			(show_name no)
+			(do_not_autoplace no)
+			(effects
+				(font
+					(size 1.27 1.27)
+				)
+				(justify right)
 			)
-			(justify left)
 		)
 	)
@@
 		(in_pos_files yes)
 		(dnp no)
-		(property "Reference" "C17"
+		(property "Reference" "C16"
 			(at 198.374 81.534 90)
 			(show_name no)
@@
 			(project "pq-register"
 				(path "/d5da316c-1ec9-4d99-8330-1c4a3f6c3ba4/f360006b-ddb2-4476-a806-4fab56f1b84d"
-					(reference "C17")
+					(reference "C16")
 					(unit 1)
 				)

Commit message: Add copyright information.
Other:
- company: (none) -> © 1962 General Precision; redrawn by Sam Hanes
Changed lines of the file:
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@@
 	(title_block
 		(title "LGP-21 P & Q Register Board")
+		(date "2026-06-15")
+		(rev "ESD 1060")
+		(company "© 1962 General Precision; redrawn by Sam Hanes")
+		(comment 1 "https://github.com/Elemecca/lgp21-docs")
 	)
 	(text "P4"
