File: boards/pq-register/Q1.kicad_sch (KiCad schematic)
At the start: 92 parts, among them Q57 T1-N652, Q58 T1-N652, Q59 T1-N652, Q60 T1-N652, Q61 T1-N652, Q62 T1-N652, Q64 T1-N652, Q66 T1-N652, Q67 T1-N652, Q68 T1-N652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

Commit message: Run ERC and clean up P & Q Register board.
Connections:
- net Q1': now reaches Q66.3 (C), R288.2, R350.1
- net ~{Q1'}: now reaches Q70.3 (C), R296.2, R362.2
Other:
- note added: "Q1"
Changed lines of the file:
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@@
 		(title "LGP-21 P & Q Register Board")
 	)
+	(text "Q1"
+		(exclude_from_sim no)
+		(at 217.17 35.56 0)
+		(effects
+			(font
+				(size 3.81 3.81)
+			)
+		)
+	)
 	(junction
 		(at 147.32 147.32)
@@
 		)
 	)
+	(label "Q1'"
+		(at 184.15 62.23 0)
+		(effects
+			(font
+				(size 1.27 1.27)
+			)
+			(justify left bottom)
+		)
+	)
+	(label "~{Q1'}"
+		(at 247.65 62.23 0)
+		(effects
+			(font
+				(size 1.27 1.27)
+			)
+			(justify left bottom)
+		)
+	)

Commit message: Add copyright information.
Other:
- company: (none) -> © 1962 General Precision; redrawn by Sam Hanes
Changed lines of the file:
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@@
 	(title_block
 		(title "LGP-21 P & Q Register Board")
+		(date "2026-06-15")
+		(rev "ESD 1060")
+		(company "© 1962 General Precision; redrawn by Sam Hanes")
+		(comment 1 "https://github.com/Elemecca/lgp21-docs")
 	)
 	(text "Q1"
